File: packages/library/american-embedded-library/libmanagement/libmanagement.kicad_pcb (KiCad board)
At the start: 0 parts

Commit message: Add Via Stitcher plugin to PCM repository
Via Stitcher is an automated via stitching and trace fencing plugin
for KiCad with Altium-style features:

- Zone Fill Mode: Fill copper zones with a grid pattern of vias
- Zone Fence Mode: Place vias around zone perimeters
- Trace Fence Mode: Shield selected traces with parallel via fences

Features:
- Configurable via size, spacing, and clearances
- Staggered or grid patterns with optional random offset
- Path-based trace fencing with smooth corner handling
- Collision detection with pads, tracks, vias, and rule areas
- Support for rounded rectangle board outlines
- Auto-preview with real-time feedback

Requires KiCad 9.0+ with IPC API support.

Co-Authored-By: Claude Opus 4.5 <noreply@anthropic.com>
Parts:
- added C1: 1uF, Capacitor_SMD:C_0402_1005Metric, F.Cu at (165.9, 74.2)
- added C2: 1uF, Capacitor_SMD:C_0402_1005Metric, F.Cu at (174.3, 74.2)
- added C3: 1uF, Capacitor_SMD:C_0402_1005Metric, F.Cu at (163.1, 74.2)
- added C4: 1uF, Capacitor_SMD:C_0402_1005Metric, F.Cu at (171.6, 74.2)
- added U1: TPS7A2018DQN, Package_SON:Texas_X2SON-4_1x1mm_P0.65mm, F.Cu at (164.5, 74.2)
- added U2: TPS7A2018DQN, Package_SON:Texas_X2SON-4_1x1mm_P0.65mm, F.Cu at (173.0, 74.2)
Routing:
- net GND: track 0.00 -> 5.61 mm, vias 0 -> 4
- net /+1V8: track 0.00 -> 1.96 mm
- net Net-(U2-IN): track 0.00 -> 0.98 mm
- net Net-(U1-IN): track 0.00 -> 0.98 mm
Other:
- copper layers 0 -> 2
